File: kicad/driva-x2.sch (KiCad schematic (older format))
At the start: 21 parts, among them J1 CONN_HALL_1, J10 CONN_SPI_2, J11 CONN_CAN, J12 CONN_POWER, J2 CONN_PROG, J3 CONN_USB_OTG, J4 CONN_SERIAL, J5 CONN_MOT_1, J6 CONN_SERVO, J7 CONN_MOT_2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

Commit message: layout and bom complete - waiting on parts from jlcpcb
Parts:
- removed J4: CONN_SERIAL, symbol Connector:Conn_01x03_Male
- removed J5: CONN_MOT_1, symbol Connector:Screw_Terminal_01x03
- removed J7: CONN_MOT_2, symbol Connector:Screw_Terminal_01x03
- added H1, H2, H3, H4: MountingHole, MountingHole:MountingHole_3.2mm_M3_Pad_Via, symbol Mechanical:MountingHole
- added H10: PAD_W_2, Connector_Wire:SolderWire-2.5sqmm_1x01_D2.4mm_OD4.4mm, symbol Mechanical:MountingHole_Pad
- added H5: PAD_U_1, Connector_Wire:SolderWire-2.5sqmm_1x01_D2.4mm_OD4.4mm, symbol Mechanical:MountingHole_Pad
- added H6: PAD_V_1, Connector_Wire:SolderWire-2.5sqmm_1x01_D2.4mm_OD4.4mm, symbol Mechanical:MountingHole_Pad
- added H7: PAD_W_1, Connector_Wire:SolderWire-2.5sqmm_1x01_D2.4mm_OD4.4mm, symbol Mechanical:MountingHole_Pad
- added H8: PAD_U_2, Connector_Wire:SolderWire-2.5sqmm_1x01_D2.4mm_OD4.4mm, symbol Mechanical:MountingHole_Pad
- added H9: PAD_V_2, Connector_Wire:SolderWire-2.5sqmm_1x01_D2.4mm_OD4.4mm, symbol Mechanical:MountingHole_Pad
- added J4: CONN_I2C, Connector_PinHeader_2.54mm:PinHeader_1x04_P2.54mm_Vertical, symbol Connector:Conn_01x04_Male
- added J5: CONN_POWER2, Connector_PinHeader_2.54mm:PinHeader_1x02_P2.54mm_Vertical, symbol Connector:Conn_01x02_Male
- J1, J2, J6, J9: footprint (none) -> Connector_PinHeader_2.54mm:PinHeader_1x05_P2.54mm_Vertical
- J10, J8: footprint (none) -> Connector_PinHeader_2.54mm:PinHeader_1x06_P2.54mm_Vertical
- J11: footprint (none) -> Connector_PinHeader_2.54mm:PinHeader_1x04_P2.54mm_Vertical
- J12: footprint (none) -> Connector_AMASS:AMASS_XT60-M_1x02_P7.20mm_Vertical; symbol Connector:Screw_Terminal_01x02 -> Connector_Generic:Conn_01x02
- J3: footprint (none) -> Connector_USB:USB_Micro-B_GCT_USB3076-30-A
- R5, R6, R8, R9: value 1k5 -> 1K5
Connections:
- net mcu/USART2_RX is gone; now on net mcu/USART1_RX: J6.3 (Pin_3)
- net mcu/USART2_TX is gone; now on net mcu/SERVO: J6.4 (Pin_4)
- net +3V3: now also J4.4 (Pin_4)
- net GND: now also J4.1 (Pin_1)
- net driver_1/OUT_U: now also H7.1
- net driver_1/OUT_V: now also H6.1
- net driver_1/OUT_W: now also H5.1
- net driver_2/OUT_U: now also H8.1
- net driver_2/OUT_V: now also H9.1
- net driver_2/OUT_W: now also H10.1
- net mcu/CAN_H: now also J11.2 (Pin_2); no longer J11.3 (Pin_3)
- net mcu/CAN_L: now also J11.3 (Pin_3); no longer J11.2 (Pin_2)
- net mcu/SERVO: no longer J6.2 (Pin_2)
- net mcu/USART1_TX: now also J6.2 (Pin_2)
- net at J3.1 (VBUS): now also J5.1 (Pin_1)
- net Power/SUPPLY renamed power/SUPPLY
- net Power/VSS renamed power/VSS
- net mcu/HALL_U_I2C_1_SCL renamed mcu/HALL_U_1
- net mcu/HALL_V_I2C_1_SDA renamed mcu/HALL_V_1
- new net ALT_POWER: J5.2 (Pin_2)
- new net mcu/I2C_1_SCL: J4.2 (Pin_2)
- new net mcu/I2C_1_SDA: J4.3 (Pin_3)
- no-connect marks 2 -> 1
Other:
- note added: "ALT_POWER is experimental. \nPlease be careful as this could fry your laptop!\n(Fuse and other protective circuits might be required)"

Commit message: Adding 0.9 version
Parts:
- removed H10: PAD_W_2, Connector_Wire:SolderWire-2.5sqmm_1x01_D2.4mm_OD4.4mm, symbol Mechanical:MountingHole_Pad
- removed H5: PAD_U_1, Connector_Wire:SolderWire-2.5sqmm_1x01_D2.4mm_OD4.4mm, symbol Mechanical:MountingHole_Pad
- removed H6: PAD_V_1, Connector_Wire:SolderWire-2.5sqmm_1x01_D2.4mm_OD4.4mm, symbol Mechanical:MountingHole_Pad
- removed H7: PAD_W_1, Connector_Wire:SolderWire-2.5sqmm_1x01_D2.4mm_OD4.4mm, symbol Mechanical:MountingHole_Pad
- removed H8: PAD_U_2, Connector_Wire:SolderWire-2.5sqmm_1x01_D2.4mm_OD4.4mm, symbol Mechanical:MountingHole_Pad
- removed H9: PAD_V_2, Connector_Wire:SolderWire-2.5sqmm_1x01_D2.4mm_OD4.4mm, symbol Mechanical:MountingHole_Pad
- removed J11: CONN_CAN, Connector_PinHeader_2.54mm:PinHeader_1x04_P2.54mm_Vertical, symbol Connector:Conn_01x04_Male
- removed J12: CONN_POWER, Connector_AMASS:AMASS_XT60-M_1x02_P7.20mm_Vertical, symbol Connector_Generic:Conn_01x02
- removed J2: CONN_PROG, Connector_PinHeader_2.54mm:PinHeader_1x05_P2.54mm_Vertical, symbol Connector:Conn_01x05_Male
- removed J4: CONN_I2C, Connector_PinHeader_2.54mm:PinHeader_1x04_P2.54mm_Vertical, symbol Connector:Conn_01x04_Male
- removed J5: CONN_POWER2, Connector_PinHeader_2.54mm:PinHeader_1x02_P2.54mm_Vertical, symbol Connector:Conn_01x02_Male
- removed J6: CONN_SERVO, Connector_PinHeader_2.54mm:PinHeader_1x05_P2.54mm_Vertical, symbol Connector:Conn_01x05_Male
- added J10: CONN_CAN, Connector_PinHeader_2.54mm:PinHeader_1x04_P2.54mm_Vertical, symbol Connector:Conn_01x04_Male
- added J11: CONN_PWR, TerminalBlock:TerminalBlock_Altech_AK300-2_P5.00mm, symbol Connector:Screw_Terminal_01x02
- added J12, J5: CONN_SERIAL, Connector_PinHeader_2.54mm:PinHeader_1x04_P2.54mm_Vertical, symbol Connector:Conn_01x04_Male
- added J2: CONN_PROG, Connector_PinHeader_2.54mm:PinHeader_1x04_P2.54mm_Vertical, symbol Connector:Conn_01x04_Male
- added J4: CONN_MOT_1, TerminalBlock:TerminalBlock_Altech_AK300-3_P5.00mm, symbol Connector:Screw_Terminal_01x03
- added J6: CONN_MOT_2, TerminalBlock:TerminalBlock_Altech_AK300-3_P5.00mm, symbol Connector:Screw_Terminal_01x03
- H1, H2, H3, H4: footprint MountingHole:MountingHole_3.2mm_M3_Pad_Via -> MountingHole:MountingHole_3.2mm_M3_ISO14580_Pad_TopBottom
- J3: footprint Connector_USB:USB_Micro-B_GCT_USB3076-30-A -> Connector_USB:USB_Micro-B_Wuerth_629105150521
- renumbered J8 to J7, J10 to J8
Connections:
- net +3V3: now also J10.4 (Pin_4), J12.4 (Pin_4), J5.4 (Pin_4)
- net GND: now also J10.1 (Pin_1), J12.1 (Pin_1), J2.3 (Pin_3), J5.1 (Pin_1)
- net mcu/CAN_H: now also J10.3 (Pin_3)
- net mcu/CAN_L: now also J10.2 (Pin_2)
- net mcu/SWCLK: now also J2.2 (Pin_2)
- net mcu/SWDIO: now also J2.4 (Pin_4)
- net mcu/USART1_RX: now also J5.3 (Pin_3)
- net mcu/USART1_TX: now also J5.2 (Pin_2)
- net power/SUPPLY: now also J11.2 (Pin_2)
- net power/VSS: now also J11.1 (Pin_1)
- net mcu/HALL_U_1 renamed mcu/HALL_U1
- net mcu/HALL_U_I2C_2_SCL renamed mcu/HALL_U2
- net mcu/HALL_V_1 renamed mcu/HALL_V1
- net mcu/HALL_V_I2C_2_SDA renamed mcu/HALL_V2
- net mcu/HALL_W_1 renamed mcu/HALL_W1
- net mcu/HALL_W_2 renamed mcu/HALL_W2
- net mcu/SPI3_MISO renamed SPI3_MOSI
- net mcu/SPI3_MOSI renamed SPI3_MISO
- net mcu/SPI3_SCLK renamed SPI3_SCLK
- new net driver-1/OUT_U: J4.3 (Pin_3)
- new net driver-1/OUT_V: J4.2 (Pin_2)
- new net driver-1/OUT_W: J4.1 (Pin_1)
- new net driver-2/OUT_U: J6.3 (Pin_3)
- new net driver-2/OUT_V: J6.2 (Pin_2)
- new net driver-2/OUT_W: J6.1 (Pin_1)
- new net imu/SCL: J12.2 (Pin_2)
- new net imu/SDA: J12.3 (Pin_3)
- new net mcu/SWO: J2.1 (Pin_1)
- no-connect marks 1 -> 2
Other:
- moved on the sheet: J9, R7, R8, R9
