File: kicad/sheet-driver.sch (KiCad schematic (older format))
At the start: 48 parts, among them Q10 TPH1R403NL, Q11 TPH1R403NL, Q12 TPH1R403NL, Q7 TPH1R403NL, Q8 TPH1R403NL, Q9 TPH1R403NL, U10 L6387ED, U11 INA240A2PW, U12 L6387ED, U7 INA240A2PW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

Commit message: layout and bom complete - waiting on parts from jlcpcb
Parts:
- added C63, C65, C67: 1n, Capacitor_SMD:C_0402_1005Metric, symbol Device:C_Small
- added C64, C66, C68: 100n, Capacitor_SMD:C_0402_1005Metric, symbol Device:C_Small
- added R62, R63, R64: 1K, Resistor_SMD:R_0402_1005Metric, symbol Device:R_Small
- C16, C21, C26: value 1uF -> 1u; footprint (none) -> Capacitor_SMD:C_0603_1608Metric
- C17, C18, C22, C23, C27, C28: value 100pF -> 100p; footprint (none) -> Capacitor_SMD:C_0402_1005Metric
- C19, C24, C29: value 470nF -> 470n; footprint (none) -> Capacitor_SMD:C_0603_1608Metric
- C20, C25, C30: value 10nF -> 10n; footprint (none) -> Capacitor_SMD:C_0402_1005Metric
- D4, D5, D6: value STPS0560Z -> b5819w; footprint (none) -> Diode_SMD:D_SOD-123
- R28, R31, R32, R34, R37, R38, R40, R43, R44: footprint (none) -> Resistor_SMD:R_0603_1608Metric
- R29, R33, R35, R39, R41, R45: footprint (none) -> Resistor_SMD:R_0402_1005Metric
- R30, R36, R42: footprint (none) -> Resistor_SMD:R_1206_3216Metric
Connections:
- net +3V3: now also C64.1, C66.1, C68.1
- net GND: now also C63.2, C64.2, C65.2, C66.2, C67.2, C68.2
- net HIN_U: no longer C18.1
- net HIN_V: no longer C23.1
- net HIN_W: no longer C28.1
- net LIN_U: now also C18.1
- net LIN_V: now also C23.1
- net LIN_W: now also C28.1
- net SENSE_U: now also C63.1, R62.1; no longer U7.8
- net SENSE_V: now also C65.1, R63.1; no longer U9.8
- net SENSE_W: now also C67.1, R64.1; no longer U11.8
- new net: R62.2, U7.8
- new net: R63.2, U9.8
- new net: R64.2, U11.8

Commit message: Adding 0.9 version
Parts:
- removed C16, C21, C26: 1u, Capacitor_SMD:C_0603_1608Metric, symbol Device:C_Small
- removed C17, C18, C22, C23, C27, C28: 100p, Capacitor_SMD:C_0402_1005Metric, symbol Device:C_Small
- removed C19, C24, C29: 470n, Capacitor_SMD:C_0603_1608Metric, symbol Device:C_Small
- removed C20, C25, C30: 10n, Capacitor_SMD:C_0402_1005Metric, symbol Device:C_Small
- removed C63, C65, C67: 1n, Capacitor_SMD:C_0402_1005Metric, symbol Device:C_Small
- removed C64, C66, C68: 100n, Capacitor_SMD:C_0402_1005Metric, symbol Device:C_Small
- removed D4, D5, D6: b5819w, Diode_SMD:D_SOD-123, symbol Device:D_Schottky_Small
- removed Q10, Q11, Q12, Q7, Q8, Q9: TPH1R403NL, Package_SO:SOP-8-1EP_4.57x4.57mm_P1.27mm_EP4.57x4.45mm_ThermalVias, symbol newo:TPH1R403NL
- removed R28, R31, R34, R37, R40, R43: 33, Resistor_SMD:R_0603_1608Metric, symbol Device:R_Small
- removed R29, R33, R35, R39, R41, R45: 10k, Resistor_SMD:R_0402_1005Metric, symbol Device:R_Small
- removed R30, R36, R42: 0.002R @1W, Resistor_SMD:R_1206_3216Metric, symbol Device:R_Small
- removed R32, R38, R44: 1, Resistor_SMD:R_0603_1608Metric, symbol Device:R_Small
- removed R62, R63, R64: 1K, Resistor_SMD:R_0402_1005Metric, symbol Device:R_Small
- removed U10, U12, U8: L6387ED, Package_SO:SOIC-8_3.9x4.9mm_P1.27mm, symbol newo:L6387ED
- removed U11, U7, U9: INA240A2PW, Package_SO:TSSOP-8_4.4x3mm_P0.65mm, symbol Amplifier_Current:INA240A2PW
Other:
- note removed: "20A peak through 0.002R = 0.04V across shunt\n50x Gain = 2.0V max on ADC\nPower in shunt = 0.04 x 20 = 0.8W"
- note removed: "PHASE_U"
- note removed: "PHASE_V"
- note removed: "PHASE_W"
